File: hardware/relojdepalabras.kicad_pcb (KiCad board)
At the start: 2 copper layers, 130 x 125 mm, 334 parts, among them J1 6P-2.54_, Q1 npn, Q10 npn, Q11 npn, Q12 npn, Q13 npn, Q14 npn, Q15 npn, Q16 npn, Q17 npn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

Commit message: primera version de pcb
Parts:
- moved R4 195.2 mm to (174.5, 33.2)
- moved R3 187.4 mm to (163.5, 33.0)
- moved R8 172.4 mm to (141.5, 33.2)
- moved R89 165.3 mm to (130.5, 33.5)
- moved R45 163.1 mm to (163.0, 70.0)
- moved R97 161.0 mm to (175.0, 94.0)
- moved R88 158.6 mm to (119.0, 33.5)
- moved U1 155.7 mm to (106.0, 33.5)
- moved R55 155.6 mm to (174.5, 106.0)
- moved R44 154.6 mm to (152.5, 70.0)
- moved R105 151.7 mm to (175.0, 118.5)
- moved R96 150.7 mm to (163.5, 94.0)
- moved R75 148.0 mm to (174.5, 130.5)
- moved R7 147.7 mm to (97.5, 33.5)
- moved R64 147.6 mm to (152.5, 82.0)
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Routing:
- net +5V: track 0.00 -> 2006.2 mm, vias 0 -> 4
- net /enable: track 0.00 -> 273.4 mm, vias 0 -> 3
- net /!sh/ld: track 0.00 -> 272.0 mm, vias 0 -> 4
- net /reloj: track 0.00 -> 182.1 mm, vias 0 -> 3
- net /datos: track 0.00 -> 135.0 mm, vias 0 -> 1
- net E/UNA: track 0.00 -> 131.0 mm, vias 0 -> 2
- net GND: track 0.00 -> 88.1 mm, vias 0 -> 12
- net Net-(R65-Pad1): track 0.00 -> 82.9 mm
- net Net-(U1-Pad9): track 0.00 -> 82.5 mm, vias 0 -> 2
- net veinte: track 0.00 -> 76.6 mm, vias 0 -> 2
- net cuarto: track 0.00 -> 76.5 mm
- net CUATRO: track 0.00 -> 76.3 mm
- net veinti: track 0.00 -> 75.9 mm
- net Net-(R34-Pad1): track 0.00 -> 71.2 mm, vias 0 -> 2
- net Net-(R66-Pad1): track 0.00 -> 70.5 mm, vias 0 -> 2
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- added copper zone on B.Cu, net GND
Other:
- rule trace_min: 0.2 -> 0.25

Commit message: agujeros de montaje metrica 4
Parts:
- added REF**: Hole_4mm, Hole_4mm, F.Cu at (175.0, 30.0)
- added REF**: Hole_4mm, Hole_4mm, F.Cu at (175.0, 145.0)
- added REF**: Hole_4mm, Hole_4mm, F.Cu at (55.0, 145.0)
- added REF**: Hole_4mm, Hole_4mm, F.Cu at (55.0, 30.0)
- moved R69 8.94 mm to (53.5, 138.5), turned to 0 degrees
- moved Q21 2.18 mm to (57.0, 140.4), turned to 270 degrees
- moved R111 2.06 mm to (175.0, 140.5)
- moved JP2 1.58 mm to (170.0, 30.0)
- moved D90 1.01 mm to (171.5, 142.5)
- moved R4 0.71 mm to (175.0, 33.7)
- moved D3 0.39 mm to (172.5, 33.5)
- moved U2 0.30 mm to (104.5, 106.1)
Routing:
- net /!sh/ld: track 272.0 -> 285.0 mm
- net GND: track 88.1 -> 99.1 mm, vias 12 -> 15
- net Net-(R69-Pad1): track 35.3 -> 24.6 mm
- net +5V: track 2006.2 -> 2016.9 mm
- net Net-(R50-Pad1): track 50.1 -> 46.2 mm
- net Net-(D90-Pad+): track 2.01 -> 4.38 mm
- net E/UNA: track 131.0 -> 132.7 mm
- net /enable: track 273.4 -> 274.2 mm
- net Net-(D3-Pad+): track 2.00 -> 2.55 mm
